File: PCB/scaarix_flow.kicad_pcb (KiCad board)
At the start: 2 copper layers, 147.6 x 146.3 mm, 56 parts

Commit message: Add files via upload
Parts:
- moved D25 7.50 mm to (84.5, 33.8), turned to -20 degrees
- moved D26 7.50 mm to (103.3, 40.6), turned to -20 degrees
- moved D1 7.50 mm to (0.00, 7.50), turned to 0 degrees
- moved D10 7.50 mm to (38.0, -18.5), turned to 0 degrees
- moved D11 7.50 mm to (38.0, -37.5), turned to 0 degrees
- moved D12 7.50 mm to (38.0, -56.5), turned to 0 degrees
- moved D13 7.50 mm to (57.0, -1.50), turned to 0 degrees
- moved D14 7.50 mm to (57.0, -20.5), turned to 0 degrees
- moved D15 7.50 mm to (57.0, -39.5), turned to 0 degrees
- moved D16 7.50 mm to (57.0, -58.5), turned to 0 degrees
- moved D17 7.50 mm to (76.0, 2.50), turned to 0 degrees
- moved D18 7.50 mm to (76.0, -16.5), turned to 0 degrees
- moved D19 7.50 mm to (76.0, -35.5), turned to 0 degrees
- moved D2 7.50 mm to (0.00, -11.5), turned to 0 degrees
- moved D20 7.50 mm to (76.0, -54.5), turned to 0 degrees
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Connections:
- D1 pad 2: P21 -> P16
- D10 pad 2: P19 -> P10
- D11 pad 2: P19 -> P6
- D12 pad 2: P19 -> P5
- D13 pad 2: P18 -> P16
- D14 pad 2: P18 -> P10
- D15 pad 2: P18 -> P6
- D16 pad 2: P18 -> P5
- D17 pad 2: P17 -> P16
- D18 pad 2: P17 -> P10
- D19 pad 2: P17 -> P6
- D2 pad 2: P21 -> P10
- D20 pad 2: P17 -> P5
- D22 pad 2: P16 -> P10
- D23 pad 2: P16 -> P6
- D24 pad 2: P16 -> P5
- D25 pad 2: P8 -> P4
- D26 pad 2: P8 -> P3
- D27 pad 2: P9 -> P3
- D3 pad 2: P21 -> P6
- D4 pad 2: P21 -> P5
- D5 pad 2: P20 -> P16
- D6 pad 2: P20 -> P10
- D7 pad 2: P20 -> P6
- D8 pad 2: P20 -> P5
- D9 pad 2: P19 -> P16
- S1 pad 2: GND -> tab_bottom
- S10 pad 2: GND -> ring_home
- S11 pad 2: GND -> ring_top
- S12 pad 2: GND -> ring_num
- S13 pad 2: GND -> middle_bottom
- S14 pad 2: GND -> middle_home
- S15 pad 2: GND -> middle_top
- S16 pad 2: GND -> middle_num
- S17 pad 1: P17 -> P15
- S17 pad 2: GND -> index_bottom
- S18 pad 1: P17 -> P15
- S18 pad 2: GND -> index_home
- S19 pad 1: P17 -> P15
- S19 pad 2: GND -> index_top
- S2 pad 2: GND -> tab_home
- S20 pad 1: P17 -> P15
- S20 pad 2: GND -> index_num
- S21 pad 1: P16 -> P14
- S21 pad 2: GND -> far_bottom
- S22 pad 1: P16 -> P14
- S22 pad 2: GND -> far_home
- S23 pad 1: P16 -> P14
- S23 pad 2: GND -> far_top
- S24 pad 1: P16 -> P14
- S24 pad 2: GND -> far_num
- S25 pad 2: GND -> 1_bottom
- S26 pad 2: GND -> 1_top
- S27 pad 2: GND -> 2_top
- S3 pad 2: GND -> tab_top
- S4 pad 2: GND -> tab_num
- S5 pad 2: GND -> pinkie_bottom
- S6 pad 2: GND -> pinkie_home
- S7 pad 2: GND -> pinkie_top
- S8 pad 2: GND -> pinkie_num
- S9 pad 2: GND -> ring_bottom
Other:
- board size 147.6 x 146.3 mm -> 147.6 x 148.8 mm
