File: PCB/scaarix_flow.kicad_pcb (KiCad board)
At the start: 2 copper layers, 147.6 x 148.8 mm, 64 parts

Commit message: Update scaarix_flow.kicad_pcb
Parts:
- removed the REF** at (87.4, 27.9)
- removed the REF** at (126.5, 67.8)
- removed the REF** at (109.7, 4.32)
- removed the REF** at (-14.7, 13.5)
- removed the REF** at (67.6, 35.3)
- removed the REF** at (106.2, 34.5)
- removed the REF** at (-14.7, -63.2)
- removed the REF** at (124.5, -62.2)
- moved MCU1 8.00 mm to (115.0, -48.0)
- moved REF** 6.00 mm to (119.5, -24.0)
Connections:
- D1 pad 1: P16 -> tab_bottom
- D12 pad 1: P5 -> ring_num
- D12 pad 2: P5 -> ring_num
- D13 pad 2: middle_bottom -> P16
- D14 pad 1: middle_home -> P10
- D15 pad 1: middle_top -> P6
- D16 pad 1: P5 -> middle_num
- D16 pad 2: middle_num -> P5
- D19 pad 1: index_top -> P6
- D2 pad 2: tab_home -> P10
- D20 pad 2: index_num -> P5
- D21 pad 1: far_bottom -> P16
- D21 pad 2: P16 -> far_bottom
- D22 pad 1: P10 -> far_home
- D24 pad 1: far_num -> P5
- D25 pad 1: P4 -> 1_bottom
- D26 pad 1: P3 -> 1_top
- D27 pad 1: 2_top -> P3
- D27 pad 2: 2_top -> P3
- D4 pad 1: tab_num -> P5
- D4 pad 2: tab_num -> P5
- D8 pad 2: pinkie_num -> P5
- D9 pad 1: ring_bottom -> P16
- D9 pad 2: P16 -> ring_bottom
Routing:
- net P18: track 201.9 -> 212.8 mm
- net P5: track 163.7 -> 153.0 mm, vias 0 -> 3
- net P4: track 120.1 -> 130.8 mm
- net P15: track 181.5 -> 192.1 mm
- net P9: track 115.5 -> 125.3 mm
- net P16: track 169.1 -> 178.6 mm
- net P6: track 152.2 -> 160.1 mm, vias 4 -> 3
- net P3: track 131.7 -> 139.6 mm
- net P19: track 224.3 -> 231.6 mm
- net P10: track 148.5 -> 155.6 mm
- net P21: track 328.5 -> 335.1 mm, vias 4 -> 6
- net P20: track 240.6 -> 247.0 mm
- net P14: track 166.4 -> 160.5 mm
- net P8: track 128.2 -> 131.4 mm
- net VCC: track 37.9 -> 35.9 mm, vias 1 -> 2
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Other:
- board size 147.6 x 148.8 mm -> 147.5 x 148.6 mm

Commit message: Update scaarix_flow.kicad_pcb
Parts:
- removed the S25 at (87.1, 26.7)
- removed the S26 at (105.9, 33.6)
- added  : , MountingHole:MountingHole_2.2mm_M2, F.Cu at (269.4, 113.6)
- added  : , MountingHole:MountingHole_2.2mm_M2, F.Cu at (130.1, 142.6)
- added  : , MountingHole:MountingHole_2.2mm_M2, F.Cu at (278.0, 208.6)
- added  : , MountingHole:MountingHole_2.2mm_M2, F.Cu at (211.4, 172.3)
- added  : , MountingHole:MountingHole_2.2mm_M2, F.Cu at (130.3, 65.2)
- added S25: , acheron_MXH:MX200H, F.Cu at (232.7, 163.1)
- added S25: , acheron_MXH:MX200H, B.Cu at (232.7, 163.1)
- added S26: , acheron_MXH:MX200H, F.Cu at (254.3, 171.0)
- added S26: , acheron_MXH:MX200H, B.Cu at (254.3, 171.0)
- S1, S10, S11, S12, S13, S14, S15, S16, S17, S18, S19, S2, S20, S21, S22, S23, S24, S27, S3, S4, S5, S6, S7, S8, S9: footprint MX -> Erics_Footprints:SW_MX_reversible
- moved S27 205.2 mm to (267.0, 197.2)
- moved D27 205.0 mm to (263.8, 204.9)
- moved REF** 200.3 mm to (272.4, 105.4)
- moved D1 194.6 mm to (145.4, 137.6)
- moved D10 194.6 mm to (183.4, 111.6)
- moved D11 194.6 mm to (183.4, 92.6)
- moved D12 194.6 mm to (183.4, 73.6)
- moved D13 194.6 mm to (202.4, 128.6)
- moved D14 194.6 mm to (202.4, 109.6)
- moved D15 194.6 mm to (202.4, 90.6)
- moved D16 194.6 mm to (202.4, 71.6)
- moved D17 194.6 mm to (221.4, 132.6)
- moved D18 194.6 mm to (221.4, 113.6)
- moved D19 194.6 mm to (221.4, 94.6)
- moved D2 194.6 mm to (145.4, 118.6)
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Connections:
- D1 pad 2: P16 -> tab_bottom
- D10 pad 1: P10 -> ring_home
- D12 pad 1: ring_num -> P5
- D13 pad 2: P16 -> middle_bottom
- D15 pad 1: P6 -> middle_top
- D16 pad 1: middle_num -> P5
- D16 pad 2: P5 -> middle_num
- D19 pad 2: P6 -> index_top
- D2 pad 2: P10 -> tab_home
- D20 pad 1: P5 -> index_num
- D20 pad 2: P5 -> index_num
- D21 pad 2: far_bottom -> P16
- D22 pad 1: far_home -> P10
- D24 pad 1: P5 -> far_num
- D24 pad 2: P5 -> far_num
- D25 pad 2: 1_bottom -> P4
- D26 pad 1: 1_top -> P3
- D3 pad 1: tab_top -> P6
- D6 pad 1: pinkie_home -> P10
- D7 pad 2: pinkie_top -> P6
- D8 pad 2: P5 -> pinkie_num
- D9 pad 1: P16 -> ring_bottom
Routing:
- net P21: track 335.1 -> 208.1 mm, vias 6 -> 12
- net P15: track 192.1 -> 114.3 mm
- net P18: track 212.8 -> 137.8 mm
- net P19: track 231.6 -> 159.4 mm, vias 4 -> 8
- net P14: track 160.5 -> 92.0 mm, vias 4 -> 2
- net P20: track 247.0 -> 184.3 mm, vias 6 -> 10
- net P4: track 130.8 -> 83.9 mm
- net P3: track 139.6 -> 180.7 mm
- net 1_bottom: track 34.3 -> 63.2 mm
- net P9: track 125.3 -> 148.4 mm
- net 1_top: track 34.3 -> 56.7 mm
- net ring_top: track 39.6 -> 18.8 mm, vias 1 -> 0
- net middle_bottom: track 39.6 -> 18.8 mm, vias 1 -> 0
- net tab_bottom: track 39.6 -> 18.8 mm, vias 1 -> 0
- net ring_bottom: track 39.6 -> 18.8 mm, vias 1 -> 0
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- added copper zone on B.Cu, net (none)
- added copper zone on F.Cu, net (none)
Other:
- board size 147.5 x 148.6 mm -> 153.4 x 160 mm
